Commit message: Enable provisional G1 waist yaw and plan bimanual teleop

File: src/hardware/bindu_description/urdf/g1_provisional.urdf (robot description, URDF)
Before this commit: robot bindu_g1_provisional, 42 links, 41 joints
Joints:
- joint leg_joint4: axis (none) -> 0 0 1; limit (none) -> lower=-1.5906 upper=1.5906 effort=30 velocity=1; type fixed -> revolute
