Commit message: fix: align Snowbot joint models with supplied URDF

File: src/hardware/bindu_description/urdf/snowbot.urdf (robot description, URDF)
Before this commit: robot snowbot, 33 links, 32 joints
Joints:
- joint arm_l_joint_6: limit lower=-1.57 upper=1.57 effort=102 velocity=4.19 -> lower=-1.309 upper=1.274 effort=102 velocity=4.19
- joint arm_l_joint_7: limit lower=-1.57 upper=1.57 effort=102 velocity=4.19 -> lower=-1.274 upper=1.449 effort=102 velocity=4.19
- joint arm_l_joint_8: limit lower=-1.57 upper=0.94 effort=42 velocity=8.59 -> lower=-1.484 upper=0.524 effort=42 velocity=8.59
- joint arm_r_joint_6: limit lower=-1.57 upper=1.57 effort=102 velocity=4.19 -> lower=-1.309 upper=1.274 effort=102 velocity=4.19
- joint arm_r_joint_7: limit lower=-1.57 upper=1.57 effort=102 velocity=4.19 -> lower=-1.274 upper=1.449 effort=102 velocity=4.19
- joint arm_r_joint_8: limit lower=-0.94 upper=1.57 effort=42 velocity=8.59 -> lower=-0.524 upper=1.484 effort=42 velocity=8.59
- joint head_joint_1: limit lower=-3.14 upper=3.14 effort=23 velocity=10.16 -> lower=-0.791 upper=0.791 effort=23 velocity=10.16
- joint head_joint_2: limit lower=-0.79 upper=0.79 effort=23 velocity=10.16 -> lower=-0.791 upper=0.791 effort=23 velocity=10.16

File: src/hardware/bindu_description/urdf/snowbot_control.urdf (robot description, URDF)
Before this commit: robot snowbot, 33 links, 32 joints
Joints:
- joint arm_l_joint_6: limit lower=-1.57 upper=1.57 effort=102 velocity=4.19 -> lower=-1.309 upper=1.274 effort=102 velocity=4.19
- joint arm_l_joint_7: limit lower=-1.57 upper=1.57 effort=102 velocity=4.19 -> lower=-1.274 upper=1.449 effort=102 velocity=4.19
- joint arm_l_joint_8: limit lower=-1.57 upper=0.94 effort=42 velocity=8.59 -> lower=-1.484 upper=0.524 effort=42 velocity=8.59
- joint arm_r_joint_6: limit lower=-1.57 upper=1.57 effort=102 velocity=4.19 -> lower=-1.309 upper=1.274 effort=102 velocity=4.19
- joint arm_r_joint_7: limit lower=-1.57 upper=1.57 effort=102 velocity=4.19 -> lower=-1.274 upper=1.449 effort=102 velocity=4.19
- joint arm_r_joint_8: limit lower=-0.94 upper=1.57 effort=42 velocity=8.59 -> lower=-0.524 upper=1.484 effort=42 velocity=8.59
- joint head_joint_1: limit lower=-3.14 upper=3.14 effort=23 velocity=10.16 -> lower=-0.791 upper=0.791 effort=23 velocity=10.16
- joint head_joint_2: limit lower=-0.79 upper=0.79 effort=23 velocity=10.16 -> lower=-0.791 upper=0.791 effort=23 velocity=10.16

File: src/hardware/bindu_description/urdf/snowbot_display.urdf (robot description, URDF)
Before this commit: robot snowbot, 33 links, 32 joints
Joints:
- joint arm_l_joint_6: limit lower=-1.57 upper=1.57 effort=102 velocity=4.19 -> lower=-1.309 upper=1.274 effort=102 velocity=4.19
- joint arm_l_joint_7: limit lower=-1.57 upper=1.57 effort=102 velocity=4.19 -> lower=-1.274 upper=1.449 effort=102 velocity=4.19
- joint arm_l_joint_8: limit lower=-1.57 upper=0.94 effort=42 velocity=8.59 -> lower=-1.484 upper=0.524 effort=42 velocity=8.59
- joint arm_r_joint_6: limit lower=-1.57 upper=1.57 effort=102 velocity=4.19 -> lower=-1.309 upper=1.274 effort=102 velocity=4.19
- joint arm_r_joint_7: limit lower=-1.57 upper=1.57 effort=102 velocity=4.19 -> lower=-1.274 upper=1.449 effort=102 velocity=4.19
- joint arm_r_joint_8: limit lower=-0.94 upper=1.57 effort=42 velocity=8.59 -> lower=-0.524 upper=1.484 effort=42 velocity=8.59
- joint head_joint_1: limit lower=-3.14 upper=3.14 effort=23 velocity=10.16 -> lower=-0.791 upper=0.791 effort=23 velocity=10.16
- joint head_joint_2: limit lower=-0.79 upper=0.79 effort=23 velocity=10.16 -> lower=-0.791 upper=0.791 effort=23 velocity=10.16
